Commit message: feat:[realsense_description] d435 description added

File: champ/champ_description/urdf/X30.urdf.xacro (robot description, xacro)
@@ -8,4 +8,5 @@
     </inertial>
   </link> -->
+  <xacro:include filename="$(find realsense2_description)/urdf/_d435.urdf.xacro" />
   <link name="TORSO">
     <inertial>
@@ -27,4 +28,9 @@
     </collision>
   </link>
+  <xacro:sensor_d435
+    parent="TORSO"
+    name="d435_camera" >
+    <origin xyz="0.1 0 0.2" rpy="0 0 0"/>
+  </xacro:sensor_d435>
   <!-- <joint name="base_joint" type="fixed">
     <parent link="base_link" />
@@ -609,5 +615,5 @@
         <argument>odom:=odom/ground_truth</argument>
       </ros>
-      <body_name>base_link</body_name>
+      <body_name>TORSO</body_name>
       <frame_name>world</frame_name>
       <update_rate>10.0</update_rate>

Commit message: feat:[champ] added imu description

File: champ/champ_description/urdf/X30.urdf.xacro (robot description, xacro)
@@ -9,4 +9,5 @@
   </link> -->
   <xacro:include filename="$(find realsense2_description)/urdf/_d435.urdf.xacro" />
+  <xacro:include filename="$(find champ_description)/urdf/imu.urdf.xacro"/>
   <link name="TORSO">
     <inertial>
@@ -28,8 +29,14 @@
     </collision>
   </link>
+  <xacro:imu_sensor xyz="0.0 0.0 0.09" rpy="0 0 0" parent="TORSO" />
   <xacro:sensor_d435
     parent="TORSO"
-    name="d435_camera" >
-    <origin xyz="0.1 0 0.2" rpy="0 0 0"/>
+    name="camera"
+    use_nominal_extrinsics="false"
+    add_plug="false"
+    use_mesh="true"
+    topics_ns="camera"
+    publish_pointcloud="true">
+  <origin xyz="0.4 0 0.12" rpy="0 0 0"/>
   </xacro:sensor_d435>
   <!-- <joint name="base_joint" type="fixed">

File: realsense2_description/urdf/_d435.urdf.xacro (robot description, xacro)
@@ -21,7 +21,8 @@
 <robot name="sensor_d435" xmlns:xacro="http://ros.org/wiki/xacro">
   <!-- Includes -->
+  <xacro:include filename="$(find realsense2_description)/urdf/_d435.gazebo.xacro"/>
   <xacro:include filename="$(find realsense2_description)/urdf/_materials.urdf.xacro" />
   <xacro:include filename="$(find realsense2_description)/urdf/_usb_plug.urdf.xacro" />
-  <xacro:macro name="sensor_d435" params="parent *origin name:=camera use_nominal_extrinsics:=false add_plug:=false use_mesh:=true">
+  <xacro:macro name="sensor_d435" params="parent *origin name:=camera use_nominal_extrinsics:=false add_plug:=false use_mesh:=true topics_ns:=camera publish_pointcloud:=true">
     <xacro:property name="M_PI" value="3.1415926535897931" />
     <!-- The following values are approximate, and the camera node
@@ -144,5 +145,7 @@
       </joint>
       <link name="${name}_color_optical_frame"/>
+      <!-- Realsense Gazebo Plugin -->
     </xacro:if>
+    <xacro:gazebo_d435 camera_name="${name}" reference_link="${name}_link" topics_ns="${topics_ns}" depth_optical_frame="${name}_depth_optical_frame" color_optical_frame="${name}_color_optical_frame" infrared1_optical_frame="${name}_left_ir_optical_frame" infrared2_optical_frame="${name}_right_ir_optical_frame" publish_pointcloud="${publish_pointcloud}"/>
     <xacro:if value="${add_plug}">
       <xacro:usb_plug parent="${name}_link" name="${name}_usb_plug">

Commit message: Added docker compose and docker file

File: champ/champ_description/urdf/X30.urdf.xacro (robot description, xacro)
@@ -10,4 +10,5 @@
   <xacro:include filename="$(find realsense2_description)/urdf/_d435.urdf.xacro" />
   <xacro:include filename="$(find champ_description)/urdf/imu.urdf.xacro"/>
+  <xacro:include filename="$(find axis_description)/urdf/axis_q62.urdf.xacro" />
   <link name="TORSO">
     <inertial>
@@ -29,9 +30,15 @@
     </collision>
   </link>
+    <!-- <xacro:axis_q62
+      prefix="payload_camera"
+      parent="TORSO"
+      topic="payload/camera/image_raw">
+      <origin xyz="0 0 0.2" rpy="0 0 0" />
+    </xacro:axis_q62> -->
   <xacro:imu_sensor xyz="0.0 0.0 0.09" rpy="0 0 0" parent="TORSO" />
   <xacro:sensor_d435
     parent="TORSO"
     name="camera"
-    use_nominal_extrinsics="false"
+    use_nominal_extrinsics="true"
     add_plug="false"
     use_mesh="true"

File: realsense2_description/urdf/_d435.gazebo.xacro (robot description, xacro)
@@ -49,11 +49,11 @@
           <horizontal_fov>${85.2*deg_to_rad}</horizontal_fov>
           <image>
-            <width>1280</width>
-            <height>720</height>
-            <format>L_INT8</format>
+            <width>640</width>
+            <height>360</height>
+            <format>RGB_INT8</format>
           </image>
           <clip>
             <near>0.1</near>
-            <far>100</far>
+            <far>90</far>
           </clip>
           <noise>
@@ -71,11 +71,11 @@
           <horizontal_fov>${85.2*deg_to_rad}</horizontal_fov>
           <image>
-            <width>1280</width>
-            <height>720</height>
-            <format>L_INT8</format>
+            <width>640</width>
+            <height>360</height>
+            <format>RGB_INT8</format>
           </image>
           <clip>
             <near>0.1</near>
-            <far>100</far>
+            <far>90</far>
           </clip>
           <noise>
@@ -93,10 +93,10 @@
           <horizontal_fov>${85.2*deg_to_rad}</horizontal_fov>
           <image>
-            <width>1280</width>
-            <height>720</height>
+            <width>640</width>
+            <height>360</height>
           </image>
           <clip>
             <near>0.1</near>
-            <far>100</far>
+            <far>90</far>
           </clip>
           <noise>

Commit message: feat:[axis_camera,x30_api] integration

File: champ/champ_description/urdf/X30.urdf.xacro (robot description, xacro)
@@ -30,10 +30,10 @@
     </collision>
   </link>
-    <!-- <xacro:axis_q62
-      prefix="payload_camera"
-      parent="TORSO"
-      topic="payload/camera/image_raw">
-      <origin xyz="0 0 0.2" rpy="0 0 0" />
-    </xacro:axis_q62> -->
+  <xacro:axis_q62
+    prefix="payload_camera"
+    parent="TORSO"
+    topic="payload/camera/image_raw">
+    <origin xyz="0 0 0.2" rpy="0 0 0" />
+  </xacro:axis_q62>
   <xacro:imu_sensor xyz="0.0 0.0 0.09" rpy="0 0 0" parent="TORSO" />
   <xacro:sensor_d435

File: champ/champ_description/urdf/imu.urdf.xacro (robot description, xacro)
@@ -32,5 +32,5 @@
     <sensor name="imu_sensor" type="imu">
         <always_on>1</always_on>
-        <update_rate>10</update_rate>
+        <update_rate>200</update_rate>
         <visualize>1</visualize>
         <topic>imu_data</topic>  <!-- Remove quotes around topic name -->
@@ -38,5 +38,5 @@
             <topicName>imu_data</topicName> <!-- Corrected syntax -->
             <bodyName>imu_sensor_link</bodyName>
-            <updateRateHZ>10.0</updateRateHZ>
+            <updateRateHZ>200</updateRateHZ>
             <gaussianNoise>0.0</gaussianNoise>
             <xyzOffset>0 0 0</xyzOffset>

Commit message: feat:[x30_ros,axis] x30 ros wrapper and tracking

File: champ/champ_description/urdf/X30.urdf.xacro (robot description, xacro)
@@ -68,7 +68,7 @@
     <parent link="TORSO" />
     <child link="FL_HIP" />
-    <axis xyz="-1 0 0" />
-    <dynamics damping="0.01" friction="0.03"/>
-    <limit lower="-0.323" upper="0.585" effort="84" velocity="17.5" />
+    <axis xyz="1 0 0" />
+    <dynamics damping="0.01" friction="0.03"/>
+    <limit lower="-0.585" upper="0.323" effort="84" velocity="17.5" />
   </joint>
   <ros2_control name="FL_HIP" type="system">
@@ -105,7 +105,7 @@
     <parent link="FL_HIP" />
     <child link="FL_THIGH" />
-    <axis xyz="0 -1 0" />
-    <dynamics damping="0.01" friction="0.03"/>
-    <limit lower="-2.967" upper="0.262" effort="84" velocity="17.5" />
+    <axis xyz="0 1 0" />
+    <dynamics damping="0.01" friction="0.03"/>
+    <limit lower="-0.262" upper="2.967" effort="84" velocity="17.5" />
   </joint>
   <ros2_control name="FL_THIGH" type="system">
@@ -154,7 +154,7 @@
     <parent link="FL_THIGH" />
     <child link="FL_SHANK" />
-    <axis xyz="0 -1 0" />
-    <dynamics damping="0.01" friction="0.03"/>
-    <limit lower="0.349" upper="2.531" effort="180" velocity="16.1" />
+    <axis xyz="0 1 0" />
+    <dynamics damping="0.01" friction="0.03"/>
+    <limit lower="-2.531" upper="-0.349" effort="180" velocity="16.1" />
   </joint>
   <ros2_control name="FL_SHANK" type="system">
@@ -211,7 +211,7 @@
     <parent link="TORSO" />
     <child link="FR_HIP" />
-    <axis xyz="-1 0 0" />
-    <dynamics damping="0.01" friction="0.03"/>
-    <limit lower="-0.585" upper="0.323" effort="84" velocity="17.5" />
+    <axis xyz="1 0 0" />
+    <dynamics damping="0.01" friction="0.03"/>
+    <limit lower="-0.323" upper="0.585" effort="84" velocity="17.5" />
   </joint>
   <ros2_control name="FR_HIP" type="system">
@@ -248,7 +248,7 @@
     <parent link="FR_HIP" />
     <child link="FR_THIGH" />
-    <axis xyz="0 -1 0" />
-    <dynamics damping="0.01" friction="0.03"/>
-    <limit lower="-2.967" upper="0.262" effort="84" velocity="17.5" />
+    <axis xyz="0 1 0" />
+    <dynamics damping="0.01" friction="0.03"/>
+    <limit lower="-0.262" upper="2.967" effort="84" velocity="17.5" />
   </joint>
   <ros2_control name="FR_THIGH" type="system">
@@ -297,7 +297,7 @@
     <parent link="FR_THIGH" />
     <child link="FR_SHANK" />
-    <axis xyz="0 -1 0" />
-    <dynamics damping="0.01" friction="0.03"/>
-    <limit lower="0.349" upper="2.531" effort="180" velocity="16.1" />
+    <axis xyz="0 1 0" />
+    <dynamics damping="0.01" friction="0.03"/>
+    <limit lower="-2.531" upper="-0.349" effort="180" velocity="16.1" />
   </joint>
   <ros2_control name="FR_SHANK" type="system">
@@ -354,7 +354,7 @@
     <parent link="TORSO" />
     <child link="HL_HIP" />
-    <axis xyz="-1 0 0" />
-    <dynamics damping="0.01" friction="0.03"/>
-    <limit lower="-0.323" upper="0.585" effort="84" velocity="17.5" />
+    <axis xyz="1 0 0" />
+    <dynamics damping="0.01" friction="0.03"/>
+    <limit lower="-0.585" upper="0.323" effort="84" velocity="17.5" />
   </joint>
   <ros2_control name="HL_HIP" type="system">
@@ -391,7 +391,7 @@
     <parent link="HL_HIP" />
     <child link="HL_THIGH" />
-    <axis xyz="0 -1 0" />
-    <dynamics damping="0.01" friction="0.03"/>
-    <limit lower="-2.967" upper="0.262" effort="84" velocity="17.5" />
+    <axis xyz="0 1 0" />
+    <dynamics damping="0.01" friction="0.03"/>
+    <limit lower="-0.262" upper="2.967" effort="84" velocity="17.5" />
   </joint>
   <ros2_control name="HL_THIGH" type="system">
@@ -440,7 +440,7 @@
     <parent link="HL_THIGH" />
     <child link="HL_SHANK" />
-    <axis xyz="0 -1 0" />
-    <dynamics damping="0.01" friction="0.03"/>
-    <limit lower="0.349" upper="2.531" effort="180" velocity="16.1" />
+    <axis xyz="0 1 0" />
+    <dynamics damping="0.01" friction="0.03"/>
+    <limit lower="-2.531" upper="-0.349" effort="180" velocity="16.1" />
   </joint>
   <ros2_control name="HL_SHANK" type="system">
@@ -497,7 +497,7 @@
     <parent link="TORSO" />
     <child link="HR_HIP" />
-    <axis xyz="-1 0 0" />
-    <dynamics damping="0.01" friction="0.03"/>
-    <limit lower="-0.585" upper="0.323" effort="84" velocity="17.5" />
+    <axis xyz="1 0 0" />
+    <dynamics damping="0.01" friction="0.03"/>
+    <limit lower="-0.323" upper="0.585" effort="84" velocity="17.5" />
   </joint>
   <ros2_control name="HR_HIP" type="system">
@@ -534,7 +534,7 @@
     <parent link="HR_HIP" />
     <child link="HR_THIGH" />
-    <axis xyz="0 -1 0" />
-    <dynamics damping="0.01" friction="0.03"/>
-    <limit lower="-2.967" upper="0.262" effort="84" velocity="17.5" />
+    <axis xyz="0 1 0" />
+    <dynamics damping="0.01" friction="0.03"/>
+    <limit lower="-0.262" upper="2.967" effort="84" velocity="17.5" />
   </joint>
   <ros2_control name="HR_THIGH" type="system">
@@ -583,7 +583,7 @@
     <parent link="HR_THIGH" />
     <child link="HR_SHANK" />
-    <axis xyz="0 -1 0" />
-    <dynamics damping="0.01" friction="0.03"/>
-    <limit lower="0.349" upper="2.531" effort="180" velocity="16.1" />
+    <axis xyz="0 1 0" />
+    <dynamics damping="0.01" friction="0.03"/>
+    <limit lower="-2.531" upper="-0.349" effort="180" velocity="16.1" />
   </joint>
   <ros2_control name="HR_SHANK" type="system">
